File: LightUpArrowHead/LightUpArrowHead.kicad_pcb (KiCad board)
At the start: 2 copper layers, 29.5 x 49 mm, 20 parts, among them J1 Conn_01x01, J2 Conn_01x01

Commit message: PCB nearly complete
Parts:
- removed D13, D14, D15, D16: D, Diode_SMD:D_SMA
- removed R3, R4, R5, R6: R_US, Resistor_SMD:R_0603_1608Metric
- added C2: Capacitor Ceramic 10uF 16V X5R 0805, Prototype Footprint - Light Up Arrow:Capacitor 0805 (Metric 2012), F.Cu at (232.0, 77.3)
- added C3: Capacitor Ceramic 10uF 16V X5R 0805, Prototype Footprint - Light Up Arrow:Capacitor 0805 (Metric 2012), F.Cu at (229.5, 80.8)
- added FID1: ~, Fiducial:Fiducial_1mm_Mask3mm, F.Cu at (216.8, 77.8)
- added FID2: ~, Fiducial:Fiducial_1mm_Mask3mm, F.Cu at (230.8, 98.3)
- added FID3: ~, Fiducial:Fiducial_1mm_Mask3mm, B.Cu at (230.3, 100.8)
- added FID4: ~, Fiducial:Fiducial_1mm_Mask3mm, B.Cu at (214.8, 76.8)
- added Q1: DMP3099L, Package_TO_SOT_SMD:SOT-23, B.Cu at (215.9, 92.3)
- added Q2: DMP3099L, Package_TO_SOT_SMD:SOT-23, B.Cu at (230.9, 92.2)
- added Q3: MOSFET N-Channel 30V 3.6A SOT-23-3, Package_TO_SOT_SMD:SOT-23, F.Cu at (215.9, 92.3)
- added Q4: MOSFET N-Channel 30V 3.6A SOT-23-3, Package_TO_SOT_SMD:SOT-23, F.Cu at (230.9, 92.2)
- C1, D1, D2, D5: moved to B.Cu
- D4: footprint Prototype Footprint - Light Up Arrow:Vishay VLD.1232G Family LED -> Prototype Footprint - Light Up Arrow:Vishay VLD.1232G Family LED - Right Angle Edge Mount (Non-Standard)
- D6: footprint Prototype Footprint - Light Up Arrow:Vishay VLD.1232G Family LED -> Prototype Footprint - Light Up Arrow:Vishay VLD.1232G Family LED - Right Angle Edge Mount (Non-Standard); moved to B.Cu
- J1, J2: value Conn_01x01 -> Edge Connector; footprint TestPoint:TestPoint_Loop_D1.80mm_Drill1.0mm_Beaded -> Prototype Footprint - Light Up Arrow:Edge Plating 3mm
- R1: value [Resistance] [Footprint] [Tolerance] -> r=3.01k; footprint Resistor_SMD:R_0402_1005Metric -> Prototype Footprint - Light Up Arrow:Resistor 0603 (Metric 1608)
- moved L1 133.7 mm to (235.3, 80.4), turned to -90 degrees
- moved R1 121.8 mm to (229.8, 77.5)
- moved D4 110.0 mm to (226.6, 63.0), turned to 0 degrees
- moved U1 108.1 mm to (232.1, 80.5), turned to 180 degrees
- moved D1 98.9 mm to (208.0, 64.0), turned to -162 degrees
- moved C1 83.6 mm to (223.4, 70.1), turned to 180 degrees
- moved D5 77.8 mm to (232.8, 63.0), turned to 180 degrees
- moved J1 75.3 mm to (217.9, 113.0)
- moved J2 74.8 mm to (228.9, 113.0)
- moved D2 73.6 mm to (214.1, 63.0), turned to 180 degrees
- moved D6 65.1 mm to (238.9, 64.0), turned to 162 degrees
- moved D3 46.8 mm to (220.3, 63.0), turned to 0 degrees
Connections:
- net Net-(U1-EN) renamed /0.5-5V
- D1 pad 2: Net-(D1-A) -> /5.5V
- D2 pad 1: Net-(D2-K) -> GND
- D2 pad 2: Net-(D1-A) -> Net-(D1-K)
- D3 pad 1: Net-(D3-K) -> GND
- D3 pad 2: Net-(D1-A) -> Net-(D3-A)
- D4 pad 1: Net-(D4-K) -> Net-(D3-A)
- D4 pad 2: Net-(D1-K) -> /5.5V
- D5 pad 2: Net-(D2-K) -> /5.5V
- D6 pad 1: Net-(D6-K) -> GND
- D6 pad 2: Net-(D3-K) -> Net-(D5-K)
- J1 pad 1: Net-(D13-K) -> /Vin+
- J2 pad 1: Net-(D15-A) -> /Vin-
- U1 pad 5: Net-(D1-A) -> /5.5V
Routing:
- net GND: track 0.00 -> 15.6 mm, vias 0 -> 9
- net /0.5-5V: track 0.00 -> 12.1 mm, vias 0 -> 4
- net /Vin-: track 0.00 -> 10.5 mm, vias 0 -> 2
- net /Vin+: track 0.00 -> 10.0 mm, vias 0 -> 2
- net Net-(U1-SW): track 0.00 -> 2.81 mm
- net Net-(U1-VSEL): track 0.00 -> 2.35 mm
- net /5.5V: track 0.00 -> 2.23 mm, vias 0 -> 1
- added copper zone on In2.Cu, net /0.5-5V
- added copper zone on F.Cu, net /Vin+
- added copper zone on B.Cu, net /Vin-
- added copper zone on In1.Cu, net GND
Other:
- board size 29.5 x 49 mm -> 36.9 x 50 mm
- copper layers 2 -> 4

Commit message: Ready to order
Parts:
- FID1, FID2, FID3, FID4: footprint Fiducial:Fiducial_1mm_Mask3mm -> Prototype Footprint - Light Up Arrow:Fiducial 1mm by 3mm
- moved FID3 2.32 mm to (230.6, 98.5)
- moved FID4 1.51 mm to (215.0, 78.3)
- moved FID1 1.06 mm to (216.1, 78.6)
- moved FID2 1.00 mm to (230.8, 97.3)
Routing:
- net /5.5V: track 2.23 -> 74.6 mm, vias 1 -> 3
- net Net-(D5-K): track 0.00 -> 8.63 mm, vias 0 -> 1
- net Net-(D3-A): track 0.00 -> 8.50 mm, vias 0 -> 1
- net Net-(D1-K): track 0.00 -> 6.70 mm, vias 0 -> 1
- net GND: track 15.6 -> 20.1 mm
- net /Vin-: track 10.5 -> 10.0 mm, vias 2 -> 3
- net /Vin+: vias 2 -> 3
Other:
- outline, holes or cut-outs redrawn
- board text added: "Light-Up Blunt Arrow Head ${RevisionPCB}"
