File: LightUpArrowHead/LightUpArrowHead.kicad_sch (KiCad schematic)
At the start: 20 parts, among them J1 Conn_01x01, J2 Conn_01x01

Commit message: PCB nearly complete
Parts:
- removed D13, D14, D15, D16: D, Diode_SMD:D_SMA, symbol Device:D
- removed J1, J2: Conn_01x01, TestPoint:TestPoint_Loop_D1.80mm_Drill1.0mm_Beaded, symbol Connector_Generic:Conn_01x01
- removed R1: [Resistance] [Footprint] [Tolerance], Resistor_SMD:R_0402_1005Metric, symbol Prototype Schematic Symbols - Light Up Arrow:Resistor 1k 0402 1%
- removed R3, R4, R5, R6: R_US, Resistor_SMD:R_0603_1608Metric, symbol Device:R_US
- added C2, C3: Capacitor Ceramic 10uF 16V X5R 0805, Prototype Footprint - Light Up Arrow:Capacitor 0805 (Metric 2012), symbol Prototype Schematic Symbols - Light Up Arrow:Capacitor Ceramic 10uF 16V X5R 0805
- added FID1, FID2, FID3, FID4: ~, Fiducial:Fiducial_1mm_Mask3mm, symbol Prototype Schematic Symbols - Light Up Arrow:Fiducial
- added J1, J2: Edge Connector, Prototype Footprint - Light Up Arrow:Edge Plating 3mm, symbol Prototype Schematic Symbols - Light Up Arrow:Edge Plating 3mm
- added Q1, Q2: DMP3099L, Package_TO_SOT_SMD:SOT-23, symbol Prototype Schematic Symbols - Light Up Arrow:MOSFET P-Channel 30V 3.8A SOT-23-3
- added Q3, Q4: MOSFET N-Channel 30V 3.6A SOT-23-3, Package_TO_SOT_SMD:SOT-23, symbol Prototype Schematic Symbols - Light Up Arrow:MOSFET N-Channel 30V 3.6A SOT-23-3
- added R1: ${SIM.PARAMS}, Prototype Footprint - Light Up Arrow:Resistor 0603 (Metric 1608), symbol Prototype Schematic Symbols - Light Up Arrow:Resistor 3.01k 0603 1%
- D2: renamed from D4; footprint Vishay VLD.1232G Family LED -> Prototype Footprint - Light Up Arrow:Vishay VLD.1232G Family LED - Right Angle Edge Mount (Non-Standard)
- D6: footprint Vishay VLD.1232G Family LED -> Prototype Footprint - Light Up Arrow:Vishay VLD.1232G Family LED - Right Angle Edge Mount (Non-Standard)
- renumbered D5 to D3, D2 to D4, D3 to D5
Connections:
- net GND: now also D2.1 (K), D3.1 (K), D6.1 (K), C2.2, C3.2, Q3.2 (S), Q4.2 (S), R1.2
- net 0.5-5V: now reaches C1.1, L1.1, U1.1 (VIN), U1.3 (EN)
- net 0.5-5V: now also C2.1, Q1.2 (S), Q2.2 (S)
- net at U1.4 (VSEL): now also R1.1
- net 5.5V: now reaches D1.2 (A), D4.2 (A), D5.2 (A), U1.5 (VOUT)
- net 5.5V: now also C3.1
- new net Vin+: J1.1 (Pin_1), Q1.3 (D), Q2.1 (G), Q3.3 (D), Q4.1 (G)
- new net Vin-: J2.1 (Pin_1), Q1.1 (G), Q2.3 (D), Q3.1 (G), Q4.3 (D)
Other:
- moved on the sheet: C1, D1, D2, D3, D4, D5, D6, L1, U1

Commit message: Ready to order
Parts:
- FID1, FID2, FID3, FID4: footprint Fiducial:Fiducial_1mm_Mask3mm -> Prototype Footprint - Light Up Arrow:Fiducial 1mm by 3mm
Changed lines of the file:
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@@
 			)
 		)
-		(property "Footprint" "Fiducial:Fiducial_1mm_Mask3mm"
+		(property "Footprint" "Prototype Footprint - Light Up Arrow:Fiducial 1mm by 3mm"
 			(at 30.48 185.42 0)
 			(effects
@@
 			)
 		)
-		(property "Footprint" "Fiducial:Fiducial_1mm_Mask3mm"
+		(property "Footprint" "Prototype Footprint - Light Up Arrow:Fiducial 1mm by 3mm"
 			(at 38.1 185.42 0)
 			(effects
@@
 			)
 		)
-		(property "Footprint" "Fiducial:Fiducial_1mm_Mask3mm"
+		(property "Footprint" "Prototype Footprint - Light Up Arrow:Fiducial 1mm by 3mm"
 			(at 38.1 193.04 0)
 			(effects
@@
 			)
 		)
-		(property "Footprint" "Fiducial:Fiducial_1mm_Mask3mm"
+		(property "Footprint" "Prototype Footprint - Light Up Arrow:Fiducial 1mm by 3mm"
 			(at 30.48 193.04 0)
 			(effects

Commit message: Ready for ordering
Parts:
- C2, C3: MPN (none) -> CL21A106KOQNNNG; Technology (none) -> SMT
- D1, D2, D3, D4, D5, D6: value LED -> LED Green (525nm) 2.9V 20mA 16000mcd SMD-2; footprint Prototype Footprint - Light Up Arrow:Vishay VLD.1232G Family LED - Right Angle Edge Mount (Non-Standard) -> Vishay VLD.1232G Family LED; MPN (none) -> VLDTG1232G-08; Technology (none) -> Handplace
- FID1, FID2, FID3, FID4: footprint Prototype Footprint - Light Up Arrow:Fiducial 1mm by 3mm -> Fiducial:Fiducial_1mm_Mask3mm
- J1, J2: now left out of the parts list
- L1: value Inductor 1uH -> Inductor 1uH 3.3A 1008; MPN (none) -> WIP252012S-1R0MLDG; Technology (none) -> SMT
- Q1, Q2: MPN (none) -> DMP3099L; Manufacturer (none) -> Diodes; Technology (none) -> SMT
- Q3, Q4: Technology (none) -> SMT
- R1: value ${SIM.PARAMS} -> Resistor 3.01k 0603 1%; MPN (none) -> RMCF0603FT3K01
- U1: value ~ -> Regulator SMPS Boost Vin=0.5-5.5V Vout=1.8-5.5V 3MHz; Technology (none) -> SMT
